Commit message: added obstacle_gazebo.xacro file and it's content
changes radar_link to lidar_link

added the  new file name to the assembler

File: src/robot_description_pkg/urdf/obstacle.urdf.xacro (robot description, xacro)
@@ -6,3 +6,4 @@
     <xacro:include filename = "material.xacro"/>
     <xacro:include filename = "obstacle_robot.xacro"/>
+    <xacro:include filename = "obstacle_gazebo.xacro"/>
 </robot>

File: src/robot_description_pkg/urdf/obstacle_robot.xacro (robot description, xacro)
@@ -15,7 +15,7 @@
 <xacro:property name ="caster_mass" value = "0.05"/>
 <xacro:property name ="caster_radius" value = "0.04"/>
-<xacro:property name ="radar_mass" value = "0.15"/>
-<xacro:property name ="radar_radius" value = "0.035"/>
-<xacro:property name ="radar_length" value = "0.04"/>
+<xacro:property name ="lidar_mass" value = "0.15"/>
+<xacro:property name ="lidar_radius" value = "0.035"/>
+<xacro:property name ="lidar_length" value = "0.04"/>
 <!--=================Inertial Xacros for the components===================-->
 <xacro:macro name = "box_inertia" params ="m l w h xyz rpy">
@@ -86,8 +86,8 @@
      h = "${box_height}" xyz = " 0 0 0 " rpy = " 0 0 0"  />
 </link>
-<link name ="radar_link">
+<link name ="lidar_link">
     <visual>
         <geometry>
-            <cylinder length = "${radar_length}" radius = "${radar_radius}"/>
+            <cylinder length = "${lidar_length}" radius = "${lidar_radius}"/>
         </geometry>
         <origin xyz = " 0 0 0" rpy = " 0 0 0"/>
@@ -96,9 +96,9 @@
     <collision>
             <geometry>
-            <cylinder length = "${radar_length}" radius = "${radar_radius}"/>
+            <cylinder length = "${lidar_length}" radius = "${lidar_radius}"/>
         </geometry>
         <origin xyz = " 0 0 0" rpy = " 0 0 0"/>
     </collision>
-    <xacro:wheel_inertia m = "${radar_mass}" r = "${radar_radius}" l = "${radar_length}"
+    <xacro:wheel_inertia m = "${lidar_mass}" r = "${lidar_radius}" l = "${lidar_length}"
     xyz = " 0 0 0 " rpy = " 0 0 0"/>
 </link>
@@ -151,8 +151,8 @@
 </joint>
 <!--Joint transforming the laser to the box_link-->
-<joint name = "box_to_radar_link" type ="fixed">
+<joint name = "box_to_lidar_link" type ="fixed">
     <parent link = "box_link"/>
-    <child link = "radar_link"/>
-    <origin xyz = "0 0 ${(box_height / 2.0) + (radar_length / 2.0)}" rpy = " 0 0 0"/>
+    <child link = "lidar_link"/>
+    <origin xyz = "0 0 ${(box_height / 2.0) + (lidar_length / 2.0)}" rpy = " 0 0 0"/>
 </joint>
 </robot>
