Commit message: Changed wheel frame trasnformation and added inertial values to the base_link frame, self_collision ignored in gazebo

File: src/robot_description_pkg/urdf/obstacle_gazebo.xacro (robot description, xacro)
@@ -1,12 +1,17 @@
 <?xml version="1.0"?>
 <robot xmlns:xacro="http://www.ros.org/wiki/xacro">
+    <gazebo reference="box_link">
+        <preserveFixedJoint>true</preserveFixedJoint> <!--Gazebo lumps all fixed joints in a single joint to preserve its physics calculation from computing physics for parts that cannot move
+        relative to each other (it normally calculates mass , inertia , collision across 6 DOF so this is a way of optimization of resources but it makes the box_link
+        frame sieze to exist which make the wheel transformation wrong  .. this is the solution telling gazebo not to lump this frame and delete it)-->
+        <material>Gazebo/Blue</material>
+        <self_collide>false</self_collide>
+    </gazebo>
     <!--Colors in gazebo(not the same as rviz)-->
-    <gazebo reference="box_link">
-        <material>Gazebo/Blue</material>
-    </gazebo>
     <gazebo reference="wheel1_link">
         <material>Gazebo/Black</material>
         <mu1>1.0</mu1> <!--Those are the coofficients of friction of the components-->
         <mu2>1.0</mu2>
+        <self_collide>false</self_collide>
     </gazebo>
     <gazebo reference="wheel2_link">
@@ -14,7 +19,9 @@
         <mu1>1.0</mu1>
         <mu2>1.0</mu2>
+        <self_collide>false</self_collide>
     </gazebo>
     <gazebo reference="lidar_link">
         <material>Gazebo/Black</material>
+        <self_collide>false</self_collide>
     </gazebo>
     <gazebo reference="caster_wheel_link">
@@ -22,13 +29,14 @@
         <mu1>0.001</mu1> <!--The riction of the caster wheel is set to a very small number to allow for sliding of the wheel-->
         <mu2>0.001</mu2>
+        <self_collide>false</self_collide>
     </gazebo>
     <!--The differential drive plugin of gazebo-->
     <gazebo>
         <plugin filename="gz-sim-diff-drive-system" name="gz::sim::systems::DiffDrive">
-            <left_joint>box_to_wheel1_link</left_joint>
-            <right_joint>box_to_wheel2_link</right_joint>
-            <wheel_separation>0.225</wheel_separation>
+            <left_joint>box_to_wheel1_joint</left_joint> <!--This is bases on the rviz visualization-->
+            <right_joint>box_to_wheel2_joint</right_joint>
+            <wheel_separation>0.21</wheel_separation>
             <wheel_radius>0.04</wheel_radius>
-            <max_wheel_torque>20</max_wheel_torque>
+            <max_wheel_torque>20</max_wheel_torque> <!--This is normally decided by the motor specs-->
             <max_wheel_acceleration>1.0</max_wheel_acceleration>
             <topic>cmd_vel</topic>
@@ -43,6 +51,6 @@
     <gazebo>
         <plugin filename="gz-sim-joint-state-publisher-system" name="gz::sim::systems::JointStatePublisher">
-            <joint_name>box_to_wheel1_link</joint_name>
-            <joint_name>box_to_wheel2_link</joint_name>
+            <joint_name>box_to_wheel1_joint</joint_name>
+            <joint_name>box_to_wheel2_joint</joint_name>
         </plugin>
     </gazebo>
@@ -86,6 +94,6 @@
             name="gz::sim::systems::JointStatePublisher">
         <topic>/world/empty/model/obstacle_robot/joint_state</topic>
-        <joint_name>box_to_wheel1_link</joint_name>
-        <joint_name>box_to_wheel2_link</joint_name>
+        <joint_name>box_to_wheel1_joint</joint_name>
+        <joint_name>box_to_wheel2_joint</joint_name>
     </plugin>
 </robot>

File: src/robot_description_pkg/urdf/obstacle_robot.xacro (robot description, xacro)
@@ -53,5 +53,5 @@
                 <cylinder length = "${wheel_length}" radius = "${wheel_radius}"/>
             </geometry>
-            <origin xyz = "0 0 0" rpy = "0 0 0"/>
+            <origin xyz = "0 0 0" rpy = "${pi / 2} 0 0"/>
             <material name = "black"/>
         </visual>
@@ -60,12 +60,17 @@
                 <cylinder length = "${wheel_length}" radius = "${wheel_radius}"/>
             </geometry>
-            <origin xyz = "0 0 0" rpy = "0 0 0"/>
+            <origin xyz = "0 0 0" rpy = "${pi / 2} 0 0"/>
         </collision>
         <xacro:wheel_inertia m = "${wheel_mass}" r = "${wheel_radius}" l = "${wheel_length}"
-        xyz = " 0 0 0 " rpy = "0 0 0 "/>
+        xyz = " 0 0 0 " rpy = "${pi/2} 0 0 "/>
     </link>
 </xacro:macro>
 <!--===============================Link Defenitions========================-->
-<link name="base_link"/>
+<link name="base_link">
+    <inertial>
+        <origin xyz = "0 0 0" rpy = " 0 0 0"/>
+        <mass value = "0.001"/>
+    </inertial>
+</link>
 <!--box link(visual / collision / inertial data)-->
 <link name ="box_link">
@@ -131,19 +136,19 @@
 </joint>
 <!--Joint to transform wheel1 to the base box_link-->
-<joint name = "box_to_wheel1_link" type = "continuous">
+<joint name = "box_to_wheel1_joint" type = "continuous">
     <parent link = "box_link"/>
     <child link = "wheel1_link"/>
-    <origin xyz = " ${box_length / 4} ${box_width / 2 + wheel_length / 2} -${box_height / 2} " rpy = " ${pi/2} 0 0"/>
-    <axis xyz="0 0 1"/>
+    <origin xyz = " ${box_length / 4} ${box_width / 2 + wheel_length / 2} -${box_height / 2} " rpy = " 0 0 0"/>
+    <axis xyz="0 1 0 "/>
 </joint>
 <!--Joint to transform the second wheel to the base_link-->
-<joint name = "box_to_wheel2_link" type  = "continuous">
+<joint name = "box_to_wheel2_joint" type  = "continuous">
     <parent link = "box_link"/>
     <child link = "wheel2_link"/>
-    <origin xyz = " ${box_length / 4} -${box_width / 2 + wheel_length / 2} -${box_height / 2}" rpy = " ${-pi / 2} 0 0 "/> <!--Because by default the cyulinder is alligned on the z-axis-->
-    <axis xyz="0 0 1"/>
+    <origin xyz = " ${box_length / 4} -${box_width / 2 + wheel_length / 2} -${box_height / 2}" rpy = " 0 0 0 "/> <!--Because by default the cyulinder is alligned on the z-axis-->
+    <axis xyz="0 1 0"/>
 </joint>
 <!--Joint transforming the caster wheel with the box_link-->
-<joint name = "box_to_caster_link" type ="fixed">
+<joint name = "box_to_caster_joint" type ="fixed">
     <parent link = "box_link"/>
     <child link = "caster_wheel_link"/>
@@ -151,5 +156,5 @@
 </joint>
 <!--Joint transforming the laser to the box_link-->
-<joint name = "box_to_lidar_link" type ="fixed">
+<joint name = "box_to_lidar_joint" type ="fixed">
     <parent link = "box_link"/>
     <child link = "lidar_link"/>
