Commit message: added the basic obstacle avoidance logic

File: src/robot_description_pkg/urdf/obstacle_robot.xacro (robot description, xacro)
@@ -68,8 +68,4 @@
 <!--===============================Link Defenitions========================-->
 <link name="base_link">
-    <inertial>
-        <origin xyz = "0 0 0" rpy = " 0 0 0"/>
-        <mass value = "0.001"/>
-    </inertial>
 </link>
 <!--box link(visual / collision / inertial data)-->
